File: pcb/allankeyboard.kicad_pcb (KiCad board)
At the start: 2 copper layers, 310 x 125 mm, 164 parts, among them U1 Nice_Nano_V2

Commit message: Finished Jounraling, added all step files and complete BOM
Connections:
- D11 pad 1: Net-(D11-K) -> Column 8
- D11 pad 2: Net-(D11-A) -> Column 8
- D12 pad 1: Net-(D12-K) -> unconnected-(D12-K-Pad1)
- D12 pad 2: Net-(D12-A) -> Column 9
- D13 pad 1: Net-(D13-K) -> Column 6
- D14 pad 1: Net-(D14-K) -> Column 7
- D25 pad 1: Net-(D25-K) -> Column 6
- D25 pad 2: Net-(D11-K) -> Column 6
- D26 pad 1: Net-(D26-K) -> Column 7
- D26 pad 2: Net-(D12-K) -> Column 7
- D27 pad 2: Net-(D13-K) -> Net-(D27-A)
- D28 pad 2: Net-(D14-K) -> Net-(D28-A)
- D40 pad 1: Net-(D40-K) -> Column 4
- D40 pad 2: Net-(D25-K) -> Column 4
- D41 pad 1: Net-(D41-K) -> Column 5
- D41 pad 2: Net-(D26-K) -> Column 5
- D42 pad 2: Net-(D27-K) -> Net-(D42-A)
- D43 pad 2: Net-(D28-K) -> Net-(D43-A)
- D44 pad 1: Net-(D44-K) -> Net-(D14-A)
- D55 pad 1: Net-(D55-K) -> Column 8
- D55 pad 2: Net-(D40-K) -> Net-(D42-K)
- D56 pad 1: Net-(D56-K) -> Column 9
- D56 pad 2: Net-(D41-K) -> Net-(D43-K)
- D57 pad 1: Net-(D57-K) -> Net-(D13-A)
- D57 pad 2: Net-(D42-K) -> Net-(D57-A)
- D58 pad 1: Column 14 -> Column 1
- D58 pad 2: Net-(D44-K) -> Column 1
- D63 pad 1: Column 4 -> Net-(D27-A)
- D64 pad 1: Column 5 -> Net-(D28-A)
- D65 pad 1: Column 6 -> Net-(D57-A)
- D66 pad 1: Column 7 -> Net-(D44-A)
- D67 pad 1: Net-(D67-K) -> Net-(D42-A)
- D68 pad 1: Net-(D68-K) -> Net-(D43-A)
- D69 pad 1: Net-(D69-K) -> Column 2
- D69 pad 2: Net-(D55-K) -> Column 2
- D70 pad 1: Net-(D70-K) -> Column 3
- D70 pad 2: Net-(D56-K) -> Column 3
- D71 pad 1: Net-(D71-K) -> Column 0
- D71 pad 2: Net-(D57-K) -> Column 0
- D72 pad 1: Column 0 -> Net-(D72-K)
- D73 pad 1: Column 1 -> Net-(D73-K)
- D74 pad 1: Column 2 -> Net-(D74-K)
- D75 pad 1: Column 3 -> Net-(D75-K)
- D76 pad 1: Column 8 -> Column 0
- D76 pad 2: Net-(D67-K) -> Net-(D72-K)
- D77 pad 1: Column 9 -> Column 1
- D77 pad 2: Net-(D68-K) -> Net-(D73-K)
- D78 pad 1: Column 10 -> Column 2
- D78 pad 2: Net-(D69-K) -> Net-(D74-K)
- D79 pad 1: Column 11 -> Column 3
- D79 pad 2: Net-(D70-K) -> Net-(D75-K)
- D80 pad 1: Column 12 -> Column 4
- D80 pad 2: Net-(D71-K) -> Net-(D27-K)
- D81 pad 1: Column 13 -> Column 5
- D81 pad 2: Net-(D43-K) -> Net-(D28-K)
- S11 pad 1: Row 0 -> Row 7
- S11 pad 2: Net-(D11-A) -> Column 8
- S12 pad 1: Row 0 -> Row 7
- S12 pad 2: Net-(D12-A) -> Column 9
- S13 pad 1: Row 0 -> Row 6
- S14 pad 1: Row 0 -> Row 6
- S25 pad 1: Row 1 -> Row 7
- S25 pad 2: Net-(D11-K) -> Column 6
- S26 pad 1: Row 1 -> Row 7
- S26 pad 2: Net-(D12-K) -> Column 7
- S27 pad 1: Row 1 -> Row 5
- S27 pad 2: Net-(D13-K) -> Net-(D27-A)
- S28 pad 1: Row 1 -> Row 5
- S28 pad 2: Net-(D14-K) -> Net-(D28-A)
- S40 pad 1: Row 2 -> Row 7
- S40 pad 2: Net-(D25-K) -> Column 4
- S41 pad 1: Row 2 -> Row 7
- S41 pad 2: Net-(D26-K) -> Column 5
- S42 pad 1: Row 2 -> Row 5
- S42 pad 2: Net-(D27-K) -> Net-(D42-A)
- S43 pad 1: Row 2 -> Row 5
- S43 pad 2: Net-(D28-K) -> Net-(D43-A)
- S44 pad 1: Row 2 -> Row 5
- S55 pad 1: Row 3 -> Row 6
- S55 pad 2: Net-(D40-K) -> Net-(D42-K)
- S56 pad 1: Row 3 -> Row 6
- S56 pad 2: Net-(D41-K) -> Net-(D43-K)
- S57 pad 1: Row 3 -> Row 5
- S57 pad 2: Net-(D42-K) -> Net-(D57-A)
- S58 pad 1: Row 3 -> Row 7
- S58 pad 2: Net-(D44-K) -> Column 1
- S69 pad 1: Row 4 -> Row 7
- S69 pad 2: Net-(D55-K) -> Column 2
- S70 pad 1: Row 4 -> Row 7
- S70 pad 2: Net-(D56-K) -> Column 3
- S71 pad 1: Row 4 -> Row 7
- S71 pad 2: Net-(D57-K) -> Column 0
- S76 pad 1: Row 5 -> Row 6
- S76 pad 2: Net-(D67-K) -> Net-(D72-K)
- S77 pad 1: Row 5 -> Row 6
- S77 pad 2: Net-(D68-K) -> Net-(D73-K)
- S78 pad 1: Row 5 -> Row 6
- S78 pad 2: Net-(D69-K) -> Net-(D74-K)
- S79 pad 1: Row 5 -> Row 6
- S79 pad 2: Net-(D70-K) -> Net-(D75-K)
- S80 pad 1: Row 5 -> Row 6
- S80 pad 2: Net-(D71-K) -> Net-(D27-K)
- S81 pad 1: Row 5 -> Row 6
- S81 pad 2: Net-(D43-K) -> Net-(D28-K)
- U1 pad 1: Row 0 -> Row 1
- U1 pad 10: Column 1 -> Row 7
- U1 pad 11: Column 2 -> Column 1
- U1 pad 12: Column 3 -> Column 0
- U1 pad 13: Column 4 -> Column 2
- U1 pad 14: Column 5 -> Column 3
- U1 pad 15: Column 6 -> Column 4
- U1 pad 16: Column 7 -> Column 5
- U1 pad 17: Column 8 -> Column 6
- U1 pad 18: Column 9 -> Column 7
- U1 pad 19: Column 10 -> Column 8
- U1 pad 2: Row 1 -> Row 0
- U1 pad 20: Column 11 -> Column 9
- U1 pad 25: Column 12 -> unconnected-(U1-1-Pad25)
- U1 pad 26: Column 13 -> unconnected-(U1-2-Pad26)
- U1 pad 27: Column 14 -> unconnected-(U1-7-Pad27)
- U1 pad 9: Column 0 -> Row 6
Routing:
- net Column 8: track 571.9 -> 151.8 mm, vias 1 -> 0
- net Row 6: track 0.00 -> 299.0 mm
- net Row 7: track 0.00 -> 292.5 mm, vias 0 -> 3
- net Column 1: track 450.6 -> 183.3 mm, vias 1 -> 0
- net Column 0: track 393.9 -> 168.0 mm, vias 0 -> 1
- net Net-(D72-K): track 0.00 -> 190.8 mm
- net Net-(D73-K): track 0.00 -> 190.6 mm
- net Net-(D28-A): track 0.00 -> 185.3 mm, vias 0 -> 1
- net Net-(D74-K): track 0.00 -> 180.9 mm
- net Column 2: track 311.5 -> 142.1 mm, vias 3 -> 2
- net Net-(D27-A): track 0.00 -> 167.6 mm, vias 0 -> 2
- net Column 11: track 158.2 -> 0.00 mm, vias 1 -> 0
- net Net-(D57-A): track 0.00 -> 157.7 mm, vias 0 -> 4
- net Net-(D44-A): track 17.9 -> 174.2 mm, vias 0 -> 1
- net Column 10: track 124.9 -> 0.00 mm, vias 3 -> 0
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